Commit message: fixed world spawning and robot spawning

File: urdf/delivery_bot/decorations.urdf.xacro (robot description, xacro)
@@ -16,5 +16,5 @@
         <origin xyz="0 0 0" rpy="0 0 0" />
         <geometry>
-          <mesh filename="package://husky_description/meshes/top_chassis.dae" />
+          <mesh filename="package://warehouse_simulation_pkg/modles/delivery_bot/top_chassis.dae" />
         </geometry>
       </visual>
@@ -30,5 +30,5 @@
         <visual>
           <geometry>
-            <mesh filename="package://husky_description/meshes/user_rail.dae" />
+            <mesh filename="package://warehouse_simulation_pkg/modles/delivery_bot/user_rail.dae" />
           </geometry>
         </visual>
@@ -45,5 +45,5 @@
       <visual>
         <geometry>
-          <mesh filename="package://husky_description/meshes/bumper.dae" />
+          <mesh filename="package://warehouse_simulation_pkg/modles/delivery_bot/bumper.dae" />
         </geometry>
       </visual>
@@ -59,5 +59,5 @@
           <visual>
               <geometry>
-                  <mesh filename="package://husky_description/meshes/bumper_extension.dae" />
+                  <mesh filename="package://warehouse_simulation_pkg/modles/delivery_bot/bumper_extension.dae" />
               </geometry>
           </visual>
@@ -73,5 +73,5 @@
       <visual>
         <geometry>
-          <mesh filename="package://husky_description/meshes/bumper.dae" />
+          <mesh filename="package://warehouse_simulation_pkg/modles/delivery_bot/bumper.dae" />
         </geometry>
       </visual>
@@ -87,5 +87,5 @@
           <visual>
               <geometry>
-                  <mesh filename="package://husky_description/meshes/bumper_extension.dae" />
+                  <mesh filename="package://warehouse_simulation_pkg/modles/delivery_bot/bumper_extension.dae" />
               </geometry>
           </visual>
@@ -104,5 +104,5 @@
             <origin xyz="0 0 0" rpy="0 0 0" />
             <geometry>
-              <mesh filename="package://husky_description/meshes/large_top_plate.dae" />
+              <mesh filename="package://warehouse_simulation_pkg/modles/delivery_bot/large_top_plate.dae" />
             </geometry>
           </visual>
@@ -110,5 +110,5 @@
             <origin xyz="0 0 0" rpy="0 0 0"/>
             <geometry>
-              <mesh filename="package://husky_description/meshes/large_top_plate_collision.stl" />
+              <mesh filename="package://warehouse_simulation_pkg/modles/delivery_bot/large_top_plate_collision.stl" />
             </geometry>
           </collision>
@@ -138,5 +138,5 @@
             <origin xyz="0 0 0" rpy="0 0 0" />
             <geometry>
-              <mesh filename="package://husky_description/meshes/top_plate.dae" />
+              <mesh filename="package://warehouse_simulation_pkg/modles/delivery_bot/top_plate.dae" />
             </geometry>
           </visual>
@@ -144,5 +144,5 @@
             <origin xyz="0 0 0" rpy="0 0 0"/>
             <geometry>
-              <mesh filename="package://husky_description/meshes/top_plate.stl" />
+              <mesh filename="package://warehouse_simulation_pkg/modles/delivery_bot/top_plate.stl" />
             </geometry>
           </collision>

File: urdf/delivery_bot/husky.urdf.xacro (robot description, xacro)
@@ -5,5 +5,5 @@
   <xacro:arg name="prefix" default="" />
   <!-- <xacro:arg name="gazebo_controllers" default="$(find husky_control)/config/control.yaml" /> -->
-  <xacro:include filename="$(find husky_description)/urdf/husky_macro.urdf.xacro" />
+  <xacro:include filename="$(find warehouse_simulation_pkg)/urdf/delivery_bot/husky_macro.urdf.xacro" />
   <!-- Load husky description -->
   <xacro:husky prefix="$(arg prefix)" />

File: urdf/delivery_bot/husky_macro.urdf.xacro (robot description, xacro)
@@ -14,9 +14,9 @@
   <xacro:arg name="urdf_extras" default="$(optenv CPR_URDF_EXTRAS empty.urdf)" />
   <!-- Included URDF/XACRO Files -->
-  <xacro:include filename="$(find husky_description)/urdf/decorations.urdf.xacro" />
-  <xacro:include filename="$(find husky_description)/urdf/wheel.urdf.xacro" />
-  <xacro:include filename="$(find husky_description)/urdf/accessories/intel_realsense.urdf.xacro"/>
-  <!-- <xacro:include filename="$(find husky_description)/urdf/accessories/sick_lms1xx_mount.urdf.xacro"/> -->
-  <xacro:include filename="$(find husky_description)/urdf/accessories/sensor_arch.urdf.xacro"/>
+  <xacro:include filename="$(find warehouse_simulation_pkg)/urdf/delivery_bot/decorations.urdf.xacro" />
+  <xacro:include filename="$(find warehouse_simulation_pkg)/urdf/delivery_bot/wheel.urdf.xacro" />
+  <xacro:include filename="$(find warehouse_simulation_pkg)/urdf/delivery_bot/accessories/intel_realsense.urdf.xacro"/>
+  <!-- <xacro:include filename="$(find warehouse_simulation_pkg)/urdf/delivery_bot/accessories/sick_lms1xx_mount.urdf.xacro"/> -->
+  <xacro:include filename="$(find warehouse_simulation_pkg)/urdf/delivery_bot/accessories/sensor_arch.urdf.xacro"/>
   <xacro:property name="M_PI" value="3.14159"/>
   <xacro:macro name="husky" params="prefix">
@@ -37,5 +37,5 @@
         <origin xyz="0 0 0" rpy="0 0 0" />
         <geometry>
-          <mesh filename="package://husky_description/meshes/base_link.dae" />
+          <mesh filename="package://warehouse_simulation_pkg/modles/delivery_bot/base_link.dae" />
         </geometry>
       </visual>

File: urdf/delivery_bot/wheel.urdf.xacro (robot description, xacro)
@@ -11,5 +11,5 @@
         <origin xyz="0 0 0" rpy="0 0 0" />
         <geometry>
-          <mesh filename="package://husky_description/meshes/wheel.dae" />
+          <mesh filename="package://warehouse_simulation_pkg/modles/delivery_bot/wheel.dae" />
         </geometry>
       </visual>

Commit message: husky appearing succesfully in custom simulation

File: urdf/delivery_bot/decorations.urdf.xacro (robot description, xacro)
@@ -8,5 +8,5 @@
   <material name="white"><color rgba="1.0 1.0 1.0 1.0" /></material>
   <material name="red"><color rgba="1.0 0.0 0.0 1.0" /></material>
-  <xacro:macro name="husky_decorate">
+  <xacro:macro name="husky_decorate" params="mesh_path">
     <xacro:property name="husky_front_bumper_extend" value="$(optenv HUSKY_FRONT_BUMPER_EXTEND 0)" />
     <xacro:property name="husky_rear_bumper_extend" value="$(optenv HUSKY_REAR_BUMPER_EXTEND 0)" />
@@ -16,6 +16,7 @@
         <origin xyz="0 0 0" rpy="0 0 0" />
         <geometry>
-          <mesh filename="package://warehouse_simulation_pkg/modles/delivery_bot/top_chassis.dae" />
+          <mesh filename="${mesh_path}top_chassis.dae" />
         </geometry>
+        <material name="black"/>
       </visual>
     </link>
@@ -30,5 +31,5 @@
         <visual>
           <geometry>
-            <mesh filename="package://warehouse_simulation_pkg/modles/delivery_bot/user_rail.dae" />
+            <mesh filename="${mesh_path}user_rail.dae" />
           </geometry>
         </visual>
@@ -45,5 +46,5 @@
       <visual>
         <geometry>
-          <mesh filename="package://warehouse_simulation_pkg/modles/delivery_bot/bumper.dae" />
+          <mesh filename="${mesh_path}bumper.dae" />
         </geometry>
       </visual>
@@ -59,5 +60,5 @@
           <visual>
               <geometry>
-                  <mesh filename="package://warehouse_simulation_pkg/modles/delivery_bot/bumper_extension.dae" />
+                  <mesh filename="${mesh_path}bumper_extension.dae" />
               </geometry>
           </visual>
@@ -73,5 +74,5 @@
       <visual>
         <geometry>
-          <mesh filename="package://warehouse_simulation_pkg/modles/delivery_bot/bumper.dae" />
+          <mesh filename="${mesh_path}bumper.dae" />
         </geometry>
       </visual>
@@ -87,5 +88,5 @@
           <visual>
               <geometry>
-                  <mesh filename="package://warehouse_simulation_pkg/modles/delivery_bot/bumper_extension.dae" />
+                  <mesh filename="${mesh_path}bumper_extension.dae" />
               </geometry>
           </visual>
@@ -104,5 +105,5 @@
             <origin xyz="0 0 0" rpy="0 0 0" />
             <geometry>
-              <mesh filename="package://warehouse_simulation_pkg/modles/delivery_bot/large_top_plate.dae" />
+              <mesh filename="${mesh_path}large_top_plate.dae" />
             </geometry>
           </visual>
@@ -110,5 +111,5 @@
             <origin xyz="0 0 0" rpy="0 0 0"/>
             <geometry>
-              <mesh filename="package://warehouse_simulation_pkg/modles/delivery_bot/large_top_plate_collision.stl" />
+              <mesh filename="${mesh_path}large_top_plate_collision.dae" />
             </geometry>
           </collision>
@@ -138,5 +139,5 @@
             <origin xyz="0 0 0" rpy="0 0 0" />
             <geometry>
-              <mesh filename="package://warehouse_simulation_pkg/modles/delivery_bot/top_plate.dae" />
+              <mesh filename="${mesh_path}top_plate.dae" />
             </geometry>
           </visual>
@@ -144,5 +145,5 @@
             <origin xyz="0 0 0" rpy="0 0 0"/>
             <geometry>
-              <mesh filename="package://warehouse_simulation_pkg/modles/delivery_bot/top_plate.stl" />
+              <mesh filename="${mesh_path}top_plate.dae" />
             </geometry>
           </collision>

File: urdf/delivery_bot/husky.urdf.xacro (robot description, xacro)
@@ -3,15 +3,19 @@
   <!-- robot name parameter -->
   <!-- <xacro:arg name="name" default="" /> -->
+  <xacro:property name="mesh_path" value="$(find warehouse_simulation_pkg)/models/delivery_bot/" />
   <xacro:arg name="prefix" default="" />
   <!-- <xacro:arg name="gazebo_controllers" default="$(find husky_control)/config/control.yaml" /> -->
   <xacro:include filename="$(find warehouse_simulation_pkg)/urdf/delivery_bot/husky_macro.urdf.xacro" />
   <!-- Load husky description -->
-  <xacro:husky prefix="$(arg prefix)" />
+  <xacro:husky prefix="$(arg prefix)" mesh_path="${mesh_path}"/>
   <xacro:if value="$(arg is_sim)">
-    <!-- <gazebo>
+    <gazebo>
       <plugin name="$(arg prefix)gazebo_ros2_control" filename="libgazebo_ros2_control.so">
-        <parameters>$(arg gazebo_controllers)</parameters>
+        <!-- <parameters>$(arg gazebo_controllers)</parameters> -->
+        <ros2_control>
+          <param>$(find warehouse_simulation_pkg)/config/empty_control.yaml</param>
+        </ros2_control>
       </plugin>
-    </gazebo> -->
+    </gazebo>
     <gazebo reference="$(arg prefix)imu_link">
       <sensor name="$(arg prefix)imu_sensor" type="imu">

File: urdf/delivery_bot/husky_macro.urdf.xacro (robot description, xacro)
@@ -20,5 +20,5 @@
   <xacro:include filename="$(find warehouse_simulation_pkg)/urdf/delivery_bot/accessories/sensor_arch.urdf.xacro"/>
   <xacro:property name="M_PI" value="3.14159"/>
-  <xacro:macro name="husky" params="prefix">
+  <xacro:macro name="husky" params="prefix mesh_path">
     <!-- Base Size -->
     <xacro:property name="base_x_size" value="0.98740000" />
@@ -37,5 +37,6 @@
         <origin xyz="0 0 0" rpy="0 0 0" />
         <geometry>
-          <mesh filename="package://warehouse_simulation_pkg/modles/delivery_bot/base_link.dae" />
+          <mesh filename="${mesh_path}base_link.dae" />
+          <!-- <box size="0.9 0.5 0.2"/> -->
         </geometry>
       </visual>
@@ -90,17 +91,17 @@
     </joint>
     <!-- Husky wheel macros -->
-    <xacro:husky_wheel wheel_prefix="${prefix}front_left">
+    <xacro:husky_wheel wheel_prefix="${prefix}front_left" mesh_path="${mesh_path}">
       <origin xyz="${wheelbase/2} ${track/2} ${wheel_vertical_offset}" rpy="0 0 0" />
     </xacro:husky_wheel>
-    <xacro:husky_wheel wheel_prefix="${prefix}front_right">
+    <xacro:husky_wheel wheel_prefix="${prefix}front_right" mesh_path="${mesh_path}">
       <origin xyz="${wheelbase/2} ${-track/2} ${wheel_vertical_offset}" rpy="0 0 0" />
     </xacro:husky_wheel>
-    <xacro:husky_wheel wheel_prefix="${prefix}rear_left">
+    <xacro:husky_wheel wheel_prefix="${prefix}rear_left" mesh_path="${mesh_path}">
       <origin xyz="${-wheelbase/2} ${track/2} ${wheel_vertical_offset}" rpy="0 0 0" />
     </xacro:husky_wheel>
-    <xacro:husky_wheel wheel_prefix="${prefix}rear_right">
+    <xacro:husky_wheel wheel_prefix="${prefix}rear_right" mesh_path="${mesh_path}">
       <origin xyz="${-wheelbase/2} ${-track/2} ${wheel_vertical_offset}" rpy="0 0 0" />
     </xacro:husky_wheel>
-    <xacro:husky_decorate />
+    <xacro:husky_decorate mesh_path="${mesh_path}"/>
     <!-- <xacro:if value="$(arg laser_enabled)">
       <xacro:sick_lms1xx_mount prefix="base"/>

File: urdf/delivery_bot/wheel.urdf.xacro (robot description, xacro)
@@ -1,5 +1,5 @@
 <?xml version="1.0"?>
 <robot xmlns:xacro="http://ros.org/wiki/xacro" name="husky_wheel">
-  <xacro:macro name="husky_wheel" params="wheel_prefix *joint_pose">
+  <xacro:macro name="husky_wheel" params="wheel_prefix mesh_path *joint_pose">
     <link name="${wheel_prefix}_wheel">
       <inertial>
@@ -11,5 +11,5 @@
         <origin xyz="0 0 0" rpy="0 0 0" />
         <geometry>
-          <mesh filename="package://warehouse_simulation_pkg/modles/delivery_bot/wheel.dae" />
+          <mesh filename="${mesh_path}wheel.dae" />
         </geometry>
       </visual>
